Commit message: added depth camera and lidar and connected to foxglove

File: src/fusion_bot/description/robot.urdf.xacro (robot description, xacro)
@@ -176,4 +176,10 @@
         <origin xyz="0.02 0 0.05" rpy="0 0 0"/> <!-- Front face of the mast -->
     </joint>
+    <link name="camera_link_optical"></link>
+    <joint name="camera_optical_joint" type="fixed">
+        <parent link="camera_link"/>
+        <child link="camera_link_optical"/>
+        <origin xyz="0 0 0" rpy="-1.5708 0 -1.5708"/>
+    </joint>
     <!-- LiDAR -->
     <link name="lidar_link">
@@ -201,6 +207,13 @@
     <!-- GAZEBO PLUGINS (DIGITAL HARDWARE)              -->
     <!-- ============================================== -->
+    <gazebo>
+        <plugin filename="gz-sim-sensors-system" name="gz::sim::systems::Sensors">
+            <render_engine>ogre2</render_engine>
+        </plugin>
+    </gazebo>
     <gazebo reference="imu_link">
         <sensor name="imu_sensor" type="imu">
+            <frame_id>imu_link</frame_id>
+            <gz_frame_id>imu_link</gz_frame_id>
             <always_on>1</always_on>
             <update_rate>100</update_rate>
@@ -211,4 +224,6 @@
     <gazebo reference="camera_link">
         <sensor name="depth_camera" type="rgbd_camera">
+            <frame_id>camera_link_optical</frame_id>
+            <gz_frame_id>camera_link_optical</gz_frame_id>
             <always_on>1</always_on>
             <update_rate>30</update_rate>
@@ -229,4 +244,6 @@
     <gazebo reference="lidar_link">
         <sensor name="lidar" type="gpu_lidar">
+            <frame_id>lidar_link</frame_id>
+            <gz_frame_id>lidar_link</gz_frame_id>
             <always_on>1</always_on>
             <update_rate>10</update_rate>
